File: devices/pico_display/rp2040zero_display.sch (EAGLE design)
At the start: 13 parts, among them U1 RP2040-ZERO'

Commit message: updates to beeper - now on main fdd board, updates to panel connectors
Parts:
- added R4: 10k, resistor:R-EU_R0603
- R1, R2: value 220R -> 1k
Connections:
- net RX_PANEL: now also R4.1
- net VCC: now also R4.2
Changed lines of the file:
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@@
 <part name="U1" library="RP2040-ZERO" deviceset="RP2040-ZERO" device="'"/>
 <part name="SV1" library="con-lstb" deviceset="MA04-1" device=""/>
-<part name="R1" library="resistor" deviceset="R-EU_" device="R0603" value="220R"/>
-<part name="R2" library="resistor" deviceset="R-EU_" device="R0603" value="220R"/>
+<part name="R1" library="resistor" deviceset="R-EU_" device="R0603" value="1k"/>
+<part name="R2" library="resistor" deviceset="R-EU_" device="R0603" value="1k"/>
 <part name="GND1" library="supply1" deviceset="GND" device=""/>
 <part name="D1" library="diode" deviceset="DIODE-" device="DO214AC" value="SK110-DIO"/>
@@
 <part name="P+3" library="supply1" deviceset="VCC" device=""/>
 <part name="P+4" library="supply1" deviceset="VCC" device=""/>
+<part name="R4" library="resistor" deviceset="R-EU_" device="R0603" value="10k"/>
+<part name="P+5" library="supply1" deviceset="VCC" device=""/>
 </parts>
 <sheets>
@@
 <instance part="P+3" gate="VCC" x="160.02" y="91.44"/>
 <instance part="P+4" gate="VCC" x="109.22" y="45.72" rot="MR90"/>
+<instance part="R4" gate="G$1" x="30.48" y="48.26" rot="R90"/>
+<instance part="P+5" gate="VCC" x="30.48" y="58.42" rot="MR0"/>
 </instances>
 <busses>
@@
 <segment>
 <pinref part="SV1" gate="1" pin="2"/>
-<wire x1="15.24" y1="38.1" x2="33.02" y2="38.1" width="0.1524" layer="91"/>
+<wire x1="15.24" y1="38.1" x2="30.48" y2="38.1" width="0.1524" layer="91"/>
 <label x="16.51" y="38.608" size="0.8128" layer="95" font="vector"/>
 <pinref part="R2" gate="G$1" pin="1"/>
+<pinref part="R4" gate="G$1" pin="1"/>
+<wire x1="30.48" y1="38.1" x2="33.02" y2="38.1" width="0.1524" layer="91"/>
+<wire x1="30.48" y1="43.18" x2="30.48" y2="38.1" width="0.1524" layer="91"/>
+<junction x="30.48" y="38.1"/>
 </segment>
 </net>
@@
 <pinref part="P+4" gate="VCC" pin="VCC"/>
 </segment>
-</net>
+<segment>
+<pinref part="R4" gate="G$1" pin="2"/>
+<pinref part="P+5" gate="VCC" pin="VCC"/>
+<wire x1="30.48" y1="53.34" x2="30.48" y2="55.88" width="0.1524" layer="91"/>
+</segment>
+</net>
