File: devices/pico_display/rp2040zero_display_buttons.brd (EAGLE design)
At the start: 38.2 x 20.6 mm, 14 parts, among them U1 RP2040-ZERO'

Commit message: fixes to display sch and brd
Parts:
- removed R3: 0R, resistor:R0603
- C1: value (none) -> 100nF
Connections:
- net GND: no longer R3.1
- net STRAP_INPUT_TYPE: no longer R3.2
Routing:
- net STRAP_INPUT_TYPE: track 18.0 -> 2.64 mm
Changed lines of the file:
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@@
 <layer number="14" name="Route14" color="1" fill="6" visible="no" active="no"/>
 <layer number="15" name="Route15" color="4" fill="6" visible="no" active="no"/>
-<layer number="16" name="Bottom" color="1" fill="1" visible="no" active="yes"/>
+<layer number="16" name="Bottom" color="1" fill="1" visible="yes" active="yes"/>
 <layer number="17" name="Pads" color="2" fill="1" visible="yes" active="yes"/>
 <layer number="18" name="Vias" color="2" fill="1" visible="yes" active="yes"/>
 <layer number="19" name="Unrouted" color="6" fill="1" visible="yes" active="yes"/>
 <layer number="20" name="Dimension" color="15" fill="1" visible="yes" active="yes"/>
-<layer number="21" name="tPlace" color="7" fill="1" visible="yes" active="yes"/>
+<layer number="21" name="tPlace" color="7" fill="1" visible="no" active="yes"/>
 <layer number="22" name="bPlace" color="7" fill="1" visible="no" active="yes"/>
-<layer number="23" name="tOrigins" color="15" fill="1" visible="yes" active="yes"/>
+<layer number="23" name="tOrigins" color="15" fill="1" visible="no" active="yes"/>
 <layer number="24" name="bOrigins" color="15" fill="1" visible="no" active="yes"/>
-<layer number="25" name="tNames" color="7" fill="1" visible="yes" active="yes"/>
+<layer number="25" name="tNames" color="7" fill="1" visible="no" active="yes"/>
 <layer number="26" name="bNames" color="7" fill="1" visible="no" active="yes"/>
-<layer number="27" name="tValues" color="7" fill="1" visible="yes" active="yes"/>
+<layer number="27" name="tValues" color="7" fill="1" visible="no" active="yes"/>
 <layer number="28" name="bValues" color="7" fill="1" visible="no" active="yes"/>
 <layer number="29" name="tStop" color="7" fill="3" visible="no" active="yes"/>
@@
 <layer number="49" name="Reference" color="7" fill="1" visible="no" active="yes"/>
 <layer number="50" name="dxf" color="7" fill="1" visible="no" active="no"/>
-<layer number="51" name="tDocu" color="7" fill="1" visible="yes" active="yes"/>
+<layer number="51" name="tDocu" color="7" fill="1" visible="no" active="yes"/>
 <layer number="52" name="bDocu" color="7" fill="1" visible="no" active="yes"/>
 <layer number="53" name="tGND_GNDA" color="7" fill="9" visible="no" active="no"/>
@@
 <element name="R2" library="resistor" package="R0603" value="1k" x="5.476875" y="12.620625" smashed="yes" rot="MR270"/>
 <element name="D1" library="diode" package="DO214AC" value="SK110-DIO" x="7.540625" y="7.46125" smashed="yes" rot="MR0"/>
-<element name="R3" library="resistor" package="R0603" value="0R" x="8.73125" y="1.190625" smashed="yes" rot="MR180"/>
 <element name="S1" library="DTSM-62N-V-B" package="DTSM62NVB" value="DTSM-62N-V-B" x="5.800625" y="4.099375" smashed="yes">
 <attribute name="TME_ELECTRONIC_COMPONENTS_PART_NUMBER" value="" x="26.120625" y="-44.160625" size="1.778" layer="27" display="off"/>
@@
 </element>
 <element name="U$1" library="OLED" package="SIP" value="OLED" x="19.129375" y="14.684375" smashed="yes"/>
-<element name="C1" library="rcl" package="C0603" value="" x="2.460625" y="8.41375" smashed="yes" rot="MR0">
+<element name="C1" library="rcl" package="C0603" value="100nF" x="2.460625" y="8.41375" smashed="yes" rot="MR0">
 <attribute name="VALUE" x="3.095625" y="6.50875" size="1.27" layer="28" rot="MR0"/>
 </element>
@@
 <contactref element="SV1" pad="4"/>
 <contactref element="U1" pad="22"/>
-<contactref element="R3" pad="1"/>
 <contactref element="S1" pad="4"/>
 <contactref element="S1" pad="3"/>
@@
 <signal name="STRAP_INPUT_TYPE">
 <contactref element="U1" pad="20"/>
-<contactref element="R3" pad="2"/>
-<wire x1="9.58125" y1="1.190625" x2="24.92375" y2="1.190625" width="0.3048" layer="16"/>
 <wire x1="24.92375" y1="1.190625" x2="25.161875" y2="1.42875" width="0.3048" layer="16"/>
 <wire x1="25.161875" y1="1.42875" x2="25.161875" y2="3.730625" width="0.3048" layer="16"/>
