File: devices/pico_display/rp2040zero_display_encoder.sch (EAGLE design)
At the start: 16 parts, among them U1 RP2040-ZERO', U2 EC12E20-24P24C-SW

Commit message: fixes to display sch and brd
Parts:
- C1: value (none) -> 100nF
- R3: value 0R -> 1k
Connections:
- net BTN_ENTER_ENC_PUSH: now also U2.S1
Changed lines of the file:
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@@
 <part name="D1" library="diode" deviceset="DIODE-" device="DO214AC" value="SK110-DIO"/>
 <part name="GND2" library="supply1" deviceset="GND" device=""/>
-<part name="R3" library="resistor" deviceset="R-EU_" device="R0603" value="0R"/>
+<part name="R3" library="resistor" deviceset="R-EU_" device="R0603" value="1k"/>
 <part name="GND3" library="supply1" deviceset="GND" device=""/>
 <part name="U$1" library="OLED" deviceset="OLED" device=""/>
@@
 <part name="P+22" library="supply1" deviceset="VCC" device=""/>
 <part name="P+1" library="supply1" deviceset="VCC" device=""/>
-<part name="C1" library="rcl" deviceset="C-EU" device="C0603"/>
+<part name="C1" library="rcl" deviceset="C-EU" device="C0603" value="100nF"/>
 <part name="R5" library="resistor" deviceset="R-EU_" device="R0603" value="2k2"/>
 <part name="R6" library="resistor" deviceset="R-EU_" device="R0603" value="2k2"/>
@@
 <label x="91.694" y="23.368" size="0.8128" layer="95" font="vector"/>
 </segment>
-</net>
+<segment>
+<pinref part="U2" gate="G$1" pin="S1"/>
+<wire x1="193.04" y1="15.24" x2="193.04" y2="25.4" width="0.1524" layer="91"/>
+<label x="192.532" y="23.368" size="0.8128" layer="95" font="vector" rot="R90"/>
+</segment>
+</net>
