File: devices/v40_pico_fdd/ce_fdd_v40.brd (EAGLE design)
At the start: 62.8 x 77 mm, 65 parts, among them IC8 TLV1117LV33DCYR, J1 USB4125-GF-A, J3 ZL231-34PG, U1 RASPBERRY_PICOSMD-TH, U11 74LVC245, U12 74LVC245, U2 74LVC245, X10 FK 03 PWN, DC connector for P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

Commit message: updates to beeper - now on main fdd board, updates to panel connectors
Parts:
- removed C3: 100 nF, rcl:C0603
- removed T1: (no value), transistor:SOT23-BEC
- added Q1: BC817-25LT3G, BC817-25LT3G:SOT96P237X111-3N
- added R37: 1k, rcl:R0603
- added S1: DTSM-62N-V-B, DTSM-62N-V-B:DTSM62NVB
- R20, R21: value 2k2 -> 10k
- R5: value 220R -> 0R
- SV2: device con-lstb:MA05-1 -> con-lstb:MA04-1
- moved R32 116.1 mm to (-12.2, -30.0)
- moved R21 114.8 mm to (-12.2, -25.1), turned to 0 degrees
- moved R20 103.6 mm to (-5.33, -14.7), turned to 0 degrees
- moved SV2 98.3 mm to (0.00, -20.6), turned to 0 degrees
- moved JP2 63.5 mm to (-10.4, -19.6), turned to 0 degrees
Connections:
- removed net ANALOG_BTNS: C3.1, R32.1, SV2.1, U1.32, U1.P$32
- removed net RX0: U1.2, U1.P$2
- removed net SCL: R21.1, SV2.3, U1.22, U1.P$22
- removed net SDA: R20.1, SV2.2, U1.21, U1.P$21
- new net BEEPER: R30.1, R31.1, U1.32, U1.P$32
- new net CAPTIVE_BTN: R20.2, S1.1, S1.2, U1.2, U1.P$2
- new net N$10: R37.2, SV2.2
- new net PANEL_RX: R32.2, U1.22, U1.P$22
- new net PANEL_TX: R37.1, U1.21, U1.P$21
- net 5V: now also R5.1, SV2.3
- net GND: now also JP2.2, Q1.2, R31.2, S1.3, S1.4, SV2.4; no longer C3.2, R5.2, SV2.5
- net N$3: now also Q1.1; no longer T1.B
- net N$4: now also LS1.2, Q1.3; no longer JP2.2, R30.1, R31.1
- net N$7: now also R5.2; no longer T1.C
- net N$9: now also R21.1, R32.1, SV2.1; no longer LS1.2, R5.1
- net STEP: no longer JP2.1
- net TX0: now also JP2.1
- net VCC: now also R20.1; no longer R20.2, R31.2, R32.2, SV2.4, T1.E
Routing:
- net SCL: track 30.8 -> 0.00 mm, vias 1 -> 0
- net PANEL_RX: track 0.00 -> 29.6 mm, vias 0 -> 1
- net BEEPER: track 0.00 -> 29.1 mm
- net ANALOG_BTNS: track 27.4 -> 0.00 mm
- net SDA: track 24.8 -> 0.00 mm
- net PANEL_TX: track 0.00 -> 23.3 mm
- net N$7: track 15.3 -> 0.00 mm
- net VCC: track 207.9 -> 198.4 mm
- net N$9: track 7.37 -> 0.00 mm
- net N$4: track 5.59 -> 0.00 mm
- net STEP: track 37.5 -> 36.0 mm
- net N$3: track 7.70 -> 6.53 mm
- net RX0: track 1.11 -> 0.00 mm
- net CAPTIVE_BTN: track 0.00 -> 1.11 mm

Commit message: changed button, added neopixel to fdd
Parts:
- added C10, C9: 100 nF, rcl:C0603
- added IC6: 74AHCT1G08GW,125, 74AHCT1G08GW_125:SOT65P212X110-5N
- added LED2: WS2812C-2020, WS2812C-2020:WS2812C2020
- added R38: 4k7, rcl:R0603
- R20: value 10k -> 1k
Connections:
- new net N$13: R20.2, S1.1, S1.2
- new net N$15: IC6.4, LED2.3
- net 5V: now also C10.1, C9.1, IC6.5, LED2.4
- net CAPTIVE_BTN: now also IC6.1, IC6.2, R38.1, S1.3, S1.4; no longer R20.2, S1.1, S1.2
- net GND: now also C10.2, C9.2, IC6.3, LED2.2, R38.2; no longer S1.3, S1.4
Changed lines of the file:
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@@
 <attribute name="TME_ELECTRONIC_COMPONENTS_PRICE-STOCK" value="" x="-1.016" y="-8.128" size="1.778" layer="27" display="off"/>
 </element>
-<element name="R20" library="rcl" package="R0603" value="10k" x="-5.334" y="-14.732"/>
+<element name="R20" library="rcl" package="R0603" value="1k" x="-5.334" y="-14.732"/>
 <element name="SV2" library="con-lstb" package="MA04-1" value="" x="0" y="-20.574">
 <attribute name="OC_NEWARK" value="unknown" x="0" y="-20.574" size="1.778" layer="27" display="off"/>
@@
 <element name="R32" library="rcl" package="R0603" value="1k" x="-12.192" y="-29.972"/>
 <element name="R37" library="rcl" package="R0603" value="1k" x="-12.192" y="-34.798"/>
+<element name="R38" library="rcl" package="R0603" value="4k7" x="-12.192" y="-39.624"/>
+<element name="C10" library="rcl" package="C0603" value="100 nF" x="-5.08" y="-44.45"/>
+<element name="LED2" library="WS2812C-2020" package="WS2812C2020" value="WS2812C-2020" x="-6.604" y="-49.022">
+<attribute name="TME_ELECTRONIC_COMPONENTS_PART_NUMBER" value="" x="-9.652" y="-49.022" size="1.778" layer="27" display="off"/>
+<attribute name="DESCRIPTION" value="Intelligent control LED integrated light source" x="-9.652" y="-49.022" size="1.778" layer="27" display="off"/>
+<attribute name="HEIGHT" value="0.84mm" x="-9.652" y="-49.022" size="1.778" layer="27" display="off"/>
+<attribute name="MANUFACTURER_NAME" value="Worldsemi" x="-9.652" y="-49.022" size="1.778" layer="27" display="off"/>
+<attribute name="MANUFACTURER_PART_NUMBER" value="WS2812C-2020" x="-9.652" y="-49.022" size="1.778" layer="27" display="off"/>
+<attribute name="TME_ELECTRONIC_COMPONENTS_PRICE-STOCK" value="" x="-9.652" y="-49.022" size="1.778" layer="27" display="off"/>
+</element>
+<element name="C9" library="rcl" package="C0603" value="100 nF" x="-12.192" y="-44.45"/>
+<element name="IC6" library="74AHCT1G08GW_125" package="SOT65P212X110-5N" value="74AHCT1G08GW,125" x="-4.064" y="-56.896">
+<attribute name="TME_ELECTRONIC_COMPONENTS_PART_NUMBER" value="" x="-15.24" y="-61.722" size="1.778" layer="27" display="off"/>
+<attribute name="DESCRIPTION" value="74AHC(T)1G08 - 2-input AND gate@en-us" x="-15.24" y="-61.722" size="1.778" layer="27" display="off"/>
+<attribute name="HEIGHT" value="1.1mm" x="-15.24" y="-61.722" size="1.778" layer="27" display="off"/>
+<attribute name="MANUFACTURER_NAME" value="Nexperia" x="-15.24" y="-61.722" size="1.778" layer="27" display="off"/>
+<attribute name="MANUFACTURER_PART_NUMBER" value="74AHCT1G08GW,125" x="-15.24" y="-61.722" size="1.778" layer="27" display="off"/>
+<attribute name="TME_ELECTRONIC_COMPONENTS_PRICE-STOCK" value="" x="-15.24" y="-61.722" size="1.778" layer="27" display="off"/>
+</element>
 </elements>
 <signals>
@@
 <wire x1="38.354" y1="38.862" x2="39.97325" y2="38.862" width="0.254" layer="1"/>
 <wire x1="39.97325" y1="38.862" x2="40.22725" y2="38.608" width="0.254" layer="1"/>
+<contactref element="R21" pad="2"/>
 <contactref element="R20" pad="1"/>
-<contactref element="R21" pad="2"/>
 <wire x1="-6.184" y1="-14.732" x2="-11.342" y2="-25.146" width="0" layer="19" extent="1-1"/>
 <wire x1="-1.666875" y1="27.178" x2="-6.184" y2="-14.732" width="0" layer="19" extent="1-1"/>
@@
 <contactref element="R31" pad="2"/>
 <contactref element="Q1" pad="2"/>
-<contactref element="S1" pad="4"/>
-<contactref element="S1" pad="3"/>
 <contactref element="SV2" pad="4"/>
 <contactref element="JP2" pad="2"/>
-<wire x1="-3.721" y1="-10.378" x2="-10.414" y2="-18.288" width="0" layer="19" extent="1-1"/>
-<wire x1="-1.05" y1="-2.987" x2="-3.721" y2="-10.378" width="0" layer="19" extent="1-1"/>
-<wire x1="4.229" y1="-10.378" x2="-3.721" y2="-10.378" width="0" layer="19" extent="1-1"/>
+<contactref element="R38" pad="2"/>
+<contactref element="C10" pad="2"/>
+<contactref element="LED2" pad="2"/>
+<contactref element="C9" pad="2"/>
+<contactref element="IC6" pad="3"/>
+<wire x1="-5.689" y1="-48.472" x2="-5.014" y2="-57.546" width="0" layer="19" extent="1-1"/>
+<wire x1="-4.23" y1="-44.45" x2="-5.689" y2="-48.472" width="0" layer="19" extent="1-1"/>
+<wire x1="-11.342" y1="-44.45" x2="-5.689" y2="-48.472" width="0" layer="19" extent="1-1"/>
+<wire x1="-11.342" y1="-39.624" x2="-11.342" y2="-44.45" width="0" layer="19" extent="1-1"/>
+<wire x1="-10.414" y1="-18.288" x2="-11.342" y2="-39.624" width="0" layer="19" extent="1-1"/>
+<wire x1="3.81" y1="-20.574" x2="-10.414" y2="-18.288" width="0" layer="19" extent="1-1"/>
+<wire x1="-1.05" y1="-2.987" x2="-10.414" y2="-18.288" width="0" layer="19" extent="1-1"/>
 <wire x1="1.27" y1="6.35" x2="-1.05" y2="-2.987" width="0" layer="19" extent="1-1"/>
-<wire x1="3.81" y1="-20.574" x2="4.229" y2="-10.378" width="0" layer="19" extent="1-1"/>
 </signal>
 <signal name="5V">
@@
 <contactref element="R5" pad="1"/>
 <contactref element="SV2" pad="3"/>
+<contactref element="C10" pad="1"/>
+<contactref element="LED2" pad="4"/>
+<contactref element="C9" pad="1"/>
+<contactref element="IC6" pad="5"/>
 <wire x1="48.28125" y1="23.443375" x2="41.656" y2="23.788" width="0" layer="19" extent="1-1"/>
 <wire x1="1.27" y1="-20.574" x2="33.274" y2="29.972" width="0" layer="19" extent="16-16"/>
+<wire x1="-5.93" y1="-44.45" x2="1.27" y2="-20.574" width="0" layer="19" extent="1-1"/>
+<wire x1="-7.519" y1="-49.572" x2="-5.93" y2="-44.45" width="0" layer="19" extent="1-1"/>
+<wire x1="-13.042" y1="-44.45" x2="-5.93" y2="-44.45" width="0" layer="19" extent="1-1"/>
+<wire x1="-3.114" y1="-56.246" x2="-7.519" y2="-49.572" width="0" layer="19" extent="1-1"/>
 </signal>
 <signal name="KEYB_RX">
@@
 </signal>
 <signal name="CAPTIVE_BTN">
-<contactref element="S1" pad="2"/>
-<contactref element="S1" pad="1"/>
-<contactref element="R20" pad="2"/>
 <contactref element="U1" pad="P$2"/>
 <contactref element="U1" pad="2"/>
 <wire x1="1.27" y1="49.182" x2="1.27" y2="50.292" width="0.254" layer="1"/>
-<wire x1="4.229" y1="-5.878" x2="1.27" y2="49.182" width="0" layer="19" extent="1-1"/>
-<wire x1="-3.721" y1="-5.878" x2="4.229" y2="-5.878" width="0" layer="19" extent="1-1"/>
-<wire x1="-4.484" y1="-14.732" x2="-3.721" y2="-5.878" width="0" layer="19" extent="1-1"/>
+<contactref element="S1" pad="4"/>
+<contactref element="R38" pad="1"/>
+<contactref element="S1" pad="3"/>
+<contactref element="IC6" pad="1"/>
+<contactref element="IC6" pad="2"/>
+<wire x1="-5.014" y1="-56.896" x2="-5.014" y2="-56.246" width="0" layer="19" extent="1-1"/>
+<wire x1="-13.042" y1="-39.624" x2="-5.014" y2="-56.246" width="0" layer="19" extent="1-1"/>
+<wire x1="-3.721" y1="-10.378" x2="-13.042" y2="-39.624" width="0" layer="19" extent="1-1"/>
+<wire x1="4.229" y1="-10.378" x2="-3.721" y2="-10.378" width="0" layer="19" extent="1-1"/>
+<wire x1="1.27" y1="49.182" x2="4.229" y2="-10.378" width="0" layer="19" extent="1-1"/>
 </signal>
 <signal name="N$9">
@@
 <wire x1="-1.27" y1="-20.574" x2="-11.342" y2="-34.798" width="0" layer="19" extent="1-1"/>
 </signal>
+<signal name="N$13">
+<contactref element="R20" pad="2"/>
+<contactref element="S1" pad="2"/>
+<contactref element="S1" pad="1"/>
+<wire x1="-3.721" y1="-5.878" x2="-4.484" y2="-14.732" width="0" layer="19" extent="1-1"/>
+<wire x1="4.229" y1="-5.878" x2="-3.721" y2="-5.878" width="0" layer="19" extent="1-1"/>
+</signal>
+<signal name="N$15">
+<contactref element="LED2" pad="3"/>
+<contactref element="IC6" pad="4"/>
+<wire x1="-7.519" y1="-48.472" x2="-3.114" y2="-57.546" width="0" layer="19" extent="1-1"/>
+</signal>
 </signals>

Commit message: fdd routed after schema changes
Parts:
- moved IC6 134.8 mm to (23.1, 75.2)
- moved LED2 128.7 mm to (27.2, 75.2)
- moved C9 127.2 mm to (23.1, 77.7), turned to 180 degrees
- moved C10 121.5 mm to (27.2, 72.6)
- moved R38 121.0 mm to (18.3, 77.5)
- moved R37 120.9 mm to (40.7, 73.9), turned to 90 degrees
- moved R32 115.2 mm to (38.6, 73.4), turned to 270 degrees
- moved R21 109.7 mm to (34.6, 74.1), turned to 180 degrees
- moved SV2 103.7 mm to (34.8, 77.2), turned to 180 degrees
- moved R20 90.8 mm to (18.3, 72.9), turned to 180 degrees
- moved S1 84.1 mm to (11.4, 75.2), turned to 180 degrees
- moved JP2 65.1 mm to (0.32, 44.6), turned to 180 degrees
- moved Q1 49.1 mm to (39.5, 27.2)
- moved C15 10.3 mm to (31.6, 74.1), turned to 180 degrees
- moved R5 5.45 mm to (44.2, 19.8), turned to 270 degrees
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Routing:
- net 5V: track 106.6 -> 193.3 mm, vias 4 -> 7
- net CAPTIVE_BTN: track 1.11 -> 62.7 mm
- net BEEPER: track 29.1 -> 85.4 mm, vias 0 -> 3
- net STEP: track 36.0 -> 9.46 mm, vias 1 -> 0
- net DSKCHG: track 48.8 -> 28.8 mm
- net PANEL_RX: track 29.6 -> 9.76 mm, vias 1 -> 0
- net RDATA: track 47.6 -> 28.0 mm
- net KEYB_TX_ORIG: track 47.5 -> 29.9 mm
- net N$7: track 0.00 -> 14.5 mm
- net VCC: track 198.4 -> 185.1 mm, vias 4 -> 5
- net PANEL_TX: track 23.3 -> 10.1 mm
- net KEYB_TX: track 43.7 -> 31.5 mm
- net N$13: track 0.00 -> 10.00 mm
- net N$4: track 0.00 -> 9.49 mm
- net N$10: track 0.00 -> 8.69 mm, vias 0 -> 1
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Other:
- board size 62.8 x 77 mm -> 62.8 x 79.2 mm
- board text added: "5V"
- board text added: "A"
- board text added: "P"
- board text added: "RX"
- board text added: "TX"
- board text added: "rev 4.04"
- board text removed: "ACT"
- board text removed: "BTNS"
- board text removed: "PWR"
- board text removed: "SCL"
- board text removed: "SDA"
- board text removed: "VCC"
- board text removed: "rev 4.03"
