File: devices/v40_pico_hdd/ce_hdd_v40.brd (EAGLE design)
At the start: 72 x 88.8 mm, 108 parts, among them IC1 74LVC373APW,118, IC11 TLV1117LV33DCYR, IC12 74LVC245AT20-13, IC2 74LVC245AT20-13, IC3 74LVC373APW,118, IC4 SN74AHCT1G125DBVR, IC5 74LVC245AT20-13, IC6 74LVC245AT20-13, IC7 74LVC245AT20-13, IC9 AZ1117H-ADJTRE1, J1 USB4125-GF-A, Q1 FDV304P, Q10 FDV304P, Q11 FDV304P, Q12 FDV304P, Q13 FDV304P, Q14 FDV304P, Q15 FDV304P, Q16 FDV304P, Q17 FDV304P, Q18 FDV304P, Q2 FDV304P, Q3 FDV304P, Q4 FDV304P, Q5 FDV304P, Q6 FDV304P, Q7 FDV304P, Q8 FDV304P, Q9 FDV304P, U1 RASPBERRY_PICOSMD-TH

Commit message: first version of merged hdd routed
Parts:
- removed C16, C17, C19: 100 nF, rcl:C0603
- added LED3: WS2812C-2020, WS2812C-2020:WS2812C2020
- C18: device rcl:C0805 -> rcl:C0603
- U$1: value RSSM1011C3BK -> SMSR-1; device RSSM1011C3BK:RSSM1011C3BK -> ce_fdd_v40:SMRS-1
- moved R21 178.5 mm to (17.8, 37.5), turned to 180 degrees
- moved R20 176.1 mm to (17.8, 38.9)
- moved R35 119.5 mm to (42.9, 30.3)
- moved R34 116.8 mm to (42.9, 31.8)
- moved C12 91.1 mm to (-35.2, 16.8)
- moved C14 91.1 mm to (-37.0, 16.7)
- moved IC11 87.3 mm to (-42.5, 19.7), turned to 180 degrees
- moved C10 85.3 mm to (-36.3, 21.2), turned to 90 degrees
- moved C18 82.9 mm to (-35.7, 27.9), turned to 90 degrees
- moved R31 82.4 mm to (-32.8, 16.5)
- moved R30 81.2 mm to (-28.3, 20.1), turned to 180 degrees
- moved C7 80.4 mm to (-44.2, 24.9)
- moved R29 79.2 mm to (-32.8, 18.0)
- moved C15 78.3 mm to (-39.9, 24.9), turned to 0 degrees
- moved U$1 62.5 mm to (-37.3, 26.9), turned to 90 degrees
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Connections:
- net 5V: now also LED3.4
- net GND: now also LED3.2; no longer C16.2, C17.2, C19.2
- net N$7: now also LED3.3
- net VCC: no longer C16.1, C17.1, C19.1
- net VCCBUS: now also C1.1, C9.1
- net VCCIO: no longer C1.1, C9.1
Routing:
- net VCC: track 120.5 -> 209.8 mm, vias 2 -> 6
- net GND: track 183.5 -> 251.2 mm, vias 22 -> 20
- net 5V: track 157.2 -> 223.2 mm, vias 6 -> 8
- net D4: track 82.3 -> 135.0 mm
- net D2: track 83.9 -> 133.6 mm, vias 1 -> 2
- net D5: track 82.1 -> 131.0 mm
- net D6: track 90.1 -> 138.0 mm, vias 3 -> 5
- net D7: track 101.1 -> 147.9 mm, vias 3 -> 5
- net OUT_LE2_RESET: track 27.7 -> 71.2 mm, vias 0 -> 2
- net 5V_IN: track 87.4 -> 45.1 mm, vias 2 -> 1
- net D1: track 69.0 -> 109.4 mm, vias 1 -> 2
- net CACK: track 41.8 -> 81.1 mm, vias 1 -> 3
- net D3: track 71.1 -> 110.3 mm
- net D0: track 74.9 -> 112.2 mm, vias 1 -> 2
- net BRESET: track 0.00 -> 31.9 mm, vias 0 -> 2
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Other:
- board size 72 x 88.8 mm -> 92.6 x 88.8 mm
- board text added: "ACSI"
- board text added: "Cosmo2ex HDD 4.04"
- board text added: "INSTALLED"
- board text added: "REMOVED"
- board text added: "SCSI"
- board text removed: "CE SCSI 4.03"

Commit message: routing finished, few tweaks done
Parts:
- removed D3: TS4148_RBG, TS4148_RBG:DIOC2012X85N
- removed IC4: SN74AHCT1G125DBVR, SN74AHCT1G125DBVR:SOT95P280X145-5N
- added D4: BAT54WSTR, BAT54WSTR:SOD2613X100N
- added IC8: 74AHCT1G08GW,125, 74AHCT1G08GW_125:SOT65P212X110-5N
- added R37, R38, R39: 10k, rcl:R0603
- added R40: 220R, rcl:R0603
- D1: value TS4148_RBG -> BAT54WSTR; device TS4148_RBG:DIOC2012X85N -> BAT54WSTR:SOD2613X100N
- moved R36 5.08 mm to (7.06, 69.8), turned to 0 degrees
- moved D1 0.32 mm to (-29.8, 12.4)
Connections:
- new net N$4: IC8.1, R40.2
- net 5V: now also IC8.5; no longer IC4.5
- net GND: now also IC8.3; no longer IC4.1, IC4.3
- net IN_OE_CS: now also R37.2
- net N$3: now also IC8.2; no longer IC4.2
- net N$7: now also IC8.4; no longer IC4.4
- net OC_INT: now also D4.2; no longer D3.2
- net OINT: now also D4.1; no longer D3.1
- net OUT_LE1_DRQ: now also R39.2
- net OUT_OE_INT: now also R38.2, R40.1
- net VCC: now also R37.1, R38.1, R39.1
Routing:
- net OUT_OE_INT: track 83.7 -> 115.1 mm, vias 3 -> 4
- net VCC: track 209.8 -> 230.3 mm, vias 6 -> 8
- net N$4: track 0.00 -> 6.28 mm
- net RST_C/D_REQ_NEOPIXEL: track 102.9 -> 97.7 mm
- net GND: track 251.2 -> 256.0 mm, vias 20 -> 21
- net N$3: track 6.44 -> 10.3 mm
- net OUT_LE1_DRQ: track 69.0 -> 72.1 mm
- net IN_OE_CS: track 70.0 -> 72.8 mm
- net KEYB_TX_ORIG: track 58.1 -> 60.0 mm
- net OC_INT: track 9.77 -> 9.18 mm
- net OC_DRQ: track 10.6 -> 10.0 mm
- net KEYB_TX: track 57.1 -> 57.6 mm, vias 0 -> 2

Commit message: pcb tidying up
Parts:
- moved SV1 55.6 mm to (32.1, 72.1), turned to 90 degrees
- moved RN5 48.7 mm to (28.6, 71.1), turned to 270 degrees
- moved R2 46.9 mm to (27.3, 67.9), turned to 270 degrees
- moved R3 46.2 mm to (27.3, 74.7), turned to 90 degrees
- moved C8 32.9 mm to (20.0, 67.6), turned to 180 degrees
- moved IC7 31.4 mm to (20.0, 72.1), turned to 180 degrees
- moved R36 1.59 mm to (5.48, 69.8)
- moved R40 1.51 mm to (5.48, 71.4)
Routing:
- net VCC: track 230.3 -> 200.3 mm, vias 8 -> 6
- net GND: track 256.0 -> 229.2 mm, vias 21 -> 67
- net KEYB_TX_ORIG: track 60.0 -> 35.8 mm
- net KEYB_RX: track 14.9 -> 35.6 mm
- net KEYB_TX: track 57.6 -> 49.1 mm, vias 2 -> 1
- net 5V: track 222.8 -> 214.5 mm
- net OUT_OE_INT: track 115.1 -> 107.2 mm
- net D2: track 133.6 -> 126.3 mm
- net CACK: track 81.1 -> 78.1 mm
- net D7: track 147.9 -> 145.4 mm
- net ACK: track 97.1 -> 94.6 mm
- net I/O: track 103.4 -> 101.3 mm
- net C/D: track 123.2 -> 121.3 mm
- net D6: track 138.0 -> 139.6 mm
- net N$3: track 10.3 -> 8.71 mm
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Other:
- board size 92.6 x 88.8 mm -> 92.8 x 89 mm

Commit message: minor components adjustment
Parts:
- C14, C15, C2, C24, C30: device rcl:C0805 -> rcl:C0603
- R18: value 470R -> 10k
Changed lines of the file:
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@@
 <element name="C13" library="rcl" package="C0603" value="100 nF" x="3.905875" y="33.774" smashed="yes" rot="R180"/>
 <element name="C6" library="rcl" package="C0603" value="100 nF" x="-15.001875" y="40.16375" smashed="yes" rot="R180"/>
-<element name="C30" library="rcl" package="C0805" value="1 uF" x="3.874125" y="31.853125" smashed="yes" rot="R180"/>
+<element name="C30" library="rcl" package="C0603" value="1 uF" x="3.874125" y="31.853125" smashed="yes" rot="R180"/>
 <element name="R14" library="rcl" package="R0603" value="5k1 (1%)" x="-36.83" y="8.651875" smashed="yes"/>
 <element name="R17" library="rcl" package="R0603" value="5k1 (1%)" x="-36.83" y="10.398125" smashed="yes"/>
 <element name="C23" library="rcl" package="C0603" value="100 nF" x="-22.24875" y="40.258375" smashed="yes" rot="R90"/>
-<element name="R18" library="rcl" package="R0603" value="470R" x="3.1195" y="73.373625" smashed="yes" rot="R270"/>
+<element name="R18" library="rcl" package="R0603" value="10k" x="3.1195" y="73.373625" smashed="yes" rot="R270"/>
 <element name="LED1" library="led" package="SML0603" value="" x="3.135375" y="76.4375" smashed="yes" rot="R90">
 <attribute name="VALUE" x="5.135375" y="75.4375" size="1.27" layer="27" rot="R90"/>
@@
 <element name="C21" library="rcl" package="C0603" value="100 nF" x="-24.765" y="26.273125" smashed="yes" rot="R180"/>
 <element name="C22" library="rcl" package="C0603" value="100 nF" x="42.06875" y="26.273125" smashed="yes" rot="R90"/>
-<element name="C2" library="rcl" package="C0805" value="1 uF" x="-23.733125" y="28.73375" smashed="yes" rot="R90"/>
-<element name="C24" library="rcl" package="C0805" value="1 uF" x="43.65625" y="26.273125" smashed="yes" rot="R90"/>
+<element name="C2" library="rcl" package="C0603" value="1 uF" x="-23.733125" y="28.73375" smashed="yes" rot="R90"/>
+<element name="C24" library="rcl" package="C0603" value="1 uF" x="43.65625" y="26.273125" smashed="yes" rot="R90"/>
 <element name="R15" library="rcl" package="R0603" value="120 R - 1%" x="7.858125" y="22.621875" smashed="yes" rot="R180"/>
 <element name="R4" library="rcl" package="R0603" value="150 R" x="7.858125" y="21.034375" smashed="yes"/>
@@
 </element>
 <element name="C12" library="rcl" package="C0603" value="100 nF" x="-35.2425" y="16.8275" smashed="yes" rot="R270"/>
-<element name="C14" library="rcl" package="C0805" value="1 uF" x="-36.98875" y="16.748125" smashed="yes" rot="R270"/>
+<element name="C14" library="rcl" package="C0603" value="1 uF" x="-36.98875" y="16.748125" smashed="yes" rot="R270"/>
 <element name="IC11" library="TLV1117LV33DCYR" package="SOT230P700X180-4N" value="TLV1117LV33DCYR" x="-42.545" y="19.685" smashed="yes" rot="R180">
 <attribute name="TME_ELECTRONIC_COMPONENTS_PART_NUMBER" value="" x="-38.1" y="19.685" size="1.778" layer="27" rot="R180" display="off"/>
@@
 <attribute name="TME_ELECTRONIC_COMPONENTS_PRICE-STOCK" value="" x="-38.1" y="19.685" size="1.778" layer="27" rot="R180" display="off"/>
 </element>
-<element name="C15" library="rcl" package="C0805" value="1 uF" x="-39.925625" y="24.92375" smashed="yes"/>
+<element name="C15" library="rcl" package="C0603" value="1 uF" x="-39.925625" y="24.92375" smashed="yes"/>
 <element name="C18" library="rcl" package="C0603" value="1 uF" x="-35.71875" y="27.94" smashed="yes" rot="R90"/>
 <element name="U$3" library="con_subd19" package="M19" value="M19" x="-25.0825" y="-3.01625" smashed="yes" rot="MR0"/>
@@
 <wire x1="-35.2425" y1="17.6775" x2="-36.195" y2="17.6775" width="0.3048" layer="1"/>
 <wire x1="-36.195" y1="17.6775" x2="-36.968125" y2="17.6775" width="0.3048" layer="1"/>
-<wire x1="-36.968125" y1="17.6775" x2="-36.98875" y2="17.698125" width="0.3048" layer="1"/>
+<wire x1="-36.968125" y1="17.6775" x2="-36.98875" y2="17.598125" width="0.3048" layer="1"/>
 <wire x1="-36.3325" y1="19.685" x2="-36.3325" y2="17.815" width="0.3048" layer="1"/>
 <wire x1="-36.3325" y1="17.815" x2="-36.195" y2="17.6775" width="0.3048" layer="1"/>
@@
 <wire x1="19.446875" y1="-2.936875" x2="20.8153" y2="-2.936875" width="0.254" layer="1"/>
 <wire x1="20.8153" y1="-2.936875" x2="22.317075" y2="-4.43865" width="0.254" layer="1"/>
-<wire x1="2.924125" y1="31.853125" x2="2.924125" y2="33.801" width="0.6096" layer="1"/>
+<wire x1="3.024125" y1="31.853125" x2="2.924125" y2="33.801" width="0.6096" layer="1"/>
 <wire x1="2.924125" y1="33.801" x2="3.055875" y2="33.774" width="0.6096" layer="1"/>
 <via x="-5.3975" y="48.10125" extent="1-16" drill="0.5" diameter="1.016"/>
@@
 <wire x1="16.748125" y1="-0.15875" x2="18.176875" y2="-1.5875" width="0.3048" layer="1"/>
 <wire x1="18.176875" y1="-1.5875" x2="18.176875" y2="-1.59385" width="0.3048" layer="1"/>
-<wire x1="-36.98875" y1="15.798125" x2="-39.37" y2="15.798125" width="0.3048" layer="1"/>
+<wire x1="-36.98875" y1="15.898125" x2="-39.37" y2="15.798125" width="0.3048" layer="1"/>
 <wire x1="-39.37" y1="15.798125" x2="-40.399375" y2="15.798125" width="0.3048" layer="1"/>
 <wire x1="-40.399375" y1="15.798125" x2="-40.863" y2="15.3345" width="0.3048" layer="1"/>
@@
 <wire x1="-25.615" y1="26.273125" x2="-25.615" y2="28.36" width="0.254" layer="1"/>
 <wire x1="-25.615" y1="28.36" x2="-24.29125" y2="29.68375" width="0.254" layer="1"/>
-<wire x1="-24.29125" y1="29.68375" x2="-23.733125" y2="29.68375" width="0.254" layer="1"/>
+<wire x1="-24.29125" y1="29.68375" x2="-23.733125" y2="29.58375" width="0.254" layer="1"/>
 <wire x1="22.317075" y1="-4.43865" x2="23.50135" y2="-3.254375" width="0.254" layer="1"/>
 <wire x1="23.50135" y1="-3.254375" x2="26.6446" y2="-3.254375" width="0.254" layer="1"/>
@@
 <wire x1="-44.688125" y1="33.908125" x2="-44.688125" y2="26.749375" width="0.6096" layer="16"/>
 <wire x1="-42.77775" y1="24.892" x2="-43.254" y2="24.92375" width="0.6096" layer="1"/>
-<wire x1="-43.254" y1="24.92375" x2="-40.875625" y2="24.92375" width="0.6096" layer="1"/>
+<wire x1="-43.254" y1="24.92375" x2="-40.775625" y2="24.92375" width="0.6096" layer="1"/>
 <wire x1="-39.395" y1="21.985" x2="-40.875625" y2="21.985" width="0.6096" layer="1"/>
-<wire x1="-40.875625" y1="21.985" x2="-40.875625" y2="24.92375" width="0.6096" layer="1"/>
+<wire x1="-40.875625" y1="21.985" x2="-40.775625" y2="24.92375" width="0.6096" layer="1"/>
 <wire x1="-44.688125" y1="26.749375" x2="-43.259375" y2="26.749375" width="0.6096" layer="16"/>
 <wire x1="-43.259375" y1="26.749375" x2="-42.941875" y2="26.67" width="0.6096" layer="16"/>
@@
 <wire x1="-23.8125" y1="24.844375" x2="-23.891875" y2="25.320625" width="0.6096" layer="16"/>
 <via x="-23.891875" y="25.320625" extent="1-16" drill="0.5" diameter="1.016"/>
-<wire x1="-23.733125" y1="27.78125" x2="-23.733125" y2="27.78375" width="0.6096" layer="1"/>
+<wire x1="-23.733125" y1="27.78125" x2="-23.733125" y2="27.88375" width="0.6096" layer="1"/>
 <wire x1="-22.24875" y1="39.408375" x2="-22.304375" y2="39.408375" width="0.3048" layer="1"/>
 <wire x1="43.495" y1="24.0198875" x2="43.495" y2="25.161875" width="0.6096" layer="1"/>
-<wire x1="43.495" y1="25.161875" x2="43.65625" y2="25.323125" width="0.6096" layer="1"/>
+<wire x1="43.495" y1="25.161875" x2="43.65625" y2="25.423125" width="0.6096" layer="1"/>
 <wire x1="43.495" y1="25.161875" x2="42.33" y2="25.161875" width="0.6096" layer="1"/>
 <wire x1="42.33" y1="25.161875" x2="42.06875" y2="25.423125" width="0.6096" layer="1"/>
@@
 <wire x1="43.4975" y1="20.855" x2="43.4975" y2="18.811875" width="0.6096" layer="1"/>
 <wire x1="43.4975" y1="18.811875" x2="43.418125" y2="18.7325" width="0.6096" layer="1"/>
-<wire x1="-23.891875" y1="27.625" x2="-23.733125" y2="27.78375" width="0.6096" layer="1"/>
+<wire x1="-23.891875" y1="27.625" x2="-23.733125" y2="27.88375" width="0.6096" layer="1"/>
 <wire x1="-23.891875" y1="27.625" x2="-23.891875" y2="26.29625" width="0.6096" layer="1"/>
 <wire x1="-23.891875" y1="26.29625" x2="-23.915" y2="26.273125" width="0.6096" layer="1"/>
@@
 </signal>
 </signals>
-<errors>
-</errors>
 </board>
 </drawing>

Commit message: components renamed, components renumbered, ACSI and SCSI variants created
Parts:
- removed C11, C12, C20: 100 nF, rcl:C0603
- removed C14, C15: 1 uF, rcl:C0603
- removed D2: SK110-DIO, diode:DO214AC
- removed IC7: 74LVC245AT20-13, 74LVC245AT20-13:SOP65P640X120-20N
- removed IC8: 74AHCT1G08GW,125, 74AHCT1G08GW_125:SOT65P212X110-5N
- removed R14, R17: 5k1 (1%), rcl:R0603
- removed R18, R37, R38, R39: 10k, rcl:R0603
- removed R36, R40: 220R, rcl:R0603
- removed RN5: DR1206-47R-4/8, resistor-net:CTS742C083
- removed SV1: (no value), con-lstb:MA04-1
- removed U1: RASPBERRY_PICOSMD-TH, RpiPico:PICO-PKG
- added C201, C204: 100 nF, rcl:C0603
- added C206, C207: 10 uF, 293D106X9016B2TE3:CAPPM3528X210N
- added C210: 1 uF, rcl:C0603
- added D102: BAT54WSTR, BAT54WSTR:SOD2613X100N
- added IC201: 74LVC245AT20-13, 74LVC245AT20-13:SOP65P640X120-20N
- added IC202, IC203: 74LVC373APW,118, 74LVC373APW_118:SOP65P640X110-20N
- added J2: USB4125-GF-A, USB4125-GF-A:USB4125GFA
- added R204, R205, R206, R207, R208, R209, R210: 110 R, rcl:R0603
- added R223: 150 R, rcl:R0603
- added RN101: DR1206-47R-4/8, resistor-net:CTS742C083
- C10, C5: value 10 uF -> 100 nF; device 293D106X9016B2TE3:CAPPM3528X210N -> rcl:C0603
- C2: value 1 uF -> 100 nF
- C6, C8: value 100 nF -> 1 uF
- D1: value BAT54WSTR -> SK110-DIO; device BAT54WSTR:SOD2613X100N -> diode:DO214AC
- IC1: value 74LVC373APW,118 -> RASPBERRY_PICOSMD-TH; device 74LVC373APW_118:SOP65P640X110-20N -> RpiPico:PICO-PKG
- IC3: value 74LVC373APW,118 -> 74LVC245AT20-13; device 74LVC373APW_118:SOP65P640X110-20N -> 74LVC245AT20-13:SOP65P640X120-20N
- IC6: value 74LVC245AT20-13 -> 74AHCT1G08GW,125; device 74LVC245AT20-13:SOP65P640X120-20N -> 74AHCT1G08GW_125:SOT65P212X110-5N
- J1: value USB4125-GF-A -> (none); device USB4125-GF-A:USB4125GFA -> con-lstb:MA04-1
- R1, R6, R7, R8: value 110 R -> 10k
- R10, R9: value 110 R -> 220R
- R3: value 10k -> 5k1 (1%)
- R4: value 150 R -> 5k1 (1%)
- R5: value 110 R -> 1k
- moved J1 98.1 mm to (32.1, 72.1), turned to 90 degrees
- moved R3 90.8 mm to (-36.8, 10.4), turned to 0 degrees
- moved D1 86.5 mm to (37.4, 66.7), turned to 180 degrees
- moved RN1 81.4 mm to (28.6, 71.1), turned to 270 degrees
- moved C8 73.6 mm to (-39.9, 24.9), turned to 0 degrees
- moved C2 65.2 mm to (41.3, 34.0)
- moved C10 65.1 mm to (-4.84, 78.2), turned to 180 degrees
- moved R5 60.0 mm to (3.12, 73.4), turned to 270 degrees
- moved C9 55.7 mm to (-2.22, 68.8), turned to 270 degrees
- moved C4 52.3 mm to (-36.3, 21.2)
- moved R9 50.0 mm to (5.48, 71.4), turned to 180 degrees
- moved R6 49.9 mm to (6.67, 66.1), turned to 270 degrees
- moved R7 49.3 mm to (4.13, 66.1), turned to 270 degrees
- moved R8 48.7 mm to (1.59, 66.1), turned to 270 degrees
- moved R10 47.2 mm to (5.48, 69.8), turned to 0 degrees
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- renumbered C13 to C202, C18 to C101, C21 to C208, C22 to C209, C23 to C205, C24 to C211, C30 to C203, D4 to D101, IC11 to IC4, IC12 to IC101, IC9 to IC204, JP1 to JP201, Q1 to Q201, Q10 to Q210, Q11 to Q211, Q12 to Q212, Q13 to Q213, Q14 to Q214, Q15 to Q215, Q16 to Q216, Q17 to Q217, Q18 to Q218, Q2 to Q202, Q3 to Q203, Q4 to Q204, Q5 to Q205, Q6 to Q206, Q7 to Q207, Q8 to Q208, Q9 to Q209, R11 to R211, R12 to R224, R13 to R212, R15 to R222, R16 to R213, R19 to R214, R20 to R125, R21 to R225, R22 to R215, R23 to R216, R24 to R217, R25 to R218, R26 to R219, R27 to R220, R28 to R221, R29 to R102, R30 to R104, R31 to R103, R32 to R202, R33 to R203, R34 to R101, R35 to R201, RN2 to RN102, RN3 to RN103, RN4 to RN104, SV2 to J203, U$1 to SW1, U$2 to J201, U$3 to J101, X1 to J202
Connections:
- net 3V3(OUT): now also IC1.36, IC1.P$36; no longer U1.36, U1.P$36
- net 5V: now also C10.1, C206.1, C8.1, C9.1, D1.A, IC6.5, R1.2; no longer C11.1, C15.1, C20.1, C4.1, D2.A, IC8.5, R3.2
- net 5V_IN: now also J2.A9, J2.B9; no longer J1.A9, J1.B9
- net AAAA: now also R204.1; no longer R1.1
- net ACK: now also IC203.17, IC203.4; no longer IC3.17, IC3.4
- net AD0: now also RN101.4; no longer RN1.4
- net AD1: now also RN101.3; no longer RN1.3
- net AD2: now also RN101.1; no longer RN1.1
- net ARESET: now also RN101.2; no longer RN1.2
- net ATN: now also IC201.6; no longer IC6.6
- net ATN_MSG: now also IC1.31, IC1.P$31, IC201.14, IC202.13, IC202.8; no longer IC1.13, IC1.8, IC6.14, U1.31, U1.P$31
- net BRESET: now also RN101.7; no longer RN1.7
- net BSY: now also IC201.5, IC202.15, IC202.6; no longer IC1.15, IC1.6, IC6.5
- net BSY_IN: now also IC201.15; no longer IC6.15
- net C/D: now also IC202.16, IC202.5; no longer IC1.16, IC1.5
- net C0: now also IC1.1, IC1.P$1; no longer U1.1, U1.P$1
- net C1: now also IC1.2, IC1.P$2; no longer U1.2, U1.P$2
- net C2: now also IC1.4, IC1.P$4; no longer U1.4, U1.P$4
- net C3: now also IC1.5, IC1.P$5; no longer U1.5, U1.P$5
- net C4: now also IC1.6, IC1.P$6, IC3.2, IC3.3; no longer IC5.2, IC5.3, U1.6, U1.P$6
- net C5: now also IC1.7, IC1.P$7, IC3.4, IC3.5; no longer IC5.4, IC5.5, U1.7, U1.P$7
- net C6: now also IC1.9, IC1.P$9, IC3.6, IC3.7; no longer IC5.6, IC5.7, U1.9, U1.P$9
- net C7: now also IC1.10, IC1.P$10, IC3.8, IC3.9; no longer IC5.8, IC5.9, U1.10, U1.P$10
- net CACK: now also IC1.14, IC1.P$14, IC203.16, IC203.5; no longer IC3.16, IC3.5, U1.14, U1.P$14
- net CKEYB_RX: now also IC5.3, R2.1, RN1.1; no longer IC7.3, R3.1, RN5.1
- net CKEYB_TX: now also IC5.16, RN1.3; no longer IC7.16, RN5.3
- net CKEYB_TX_ORIG: now also IC5.2, R1.1, RN1.4; no longer IC7.2, R2.1, RN5.4
- net D0: now also R204.2, RN101.5; no longer R1.2, RN1.5
- net D1: now also R205.2, RN101.6; no longer R5.2, RN1.6
- net D2: now also R206.2, RN101.8; no longer R6.2, RN1.8
- net D3: now also R207.2; no longer R7.2
- net D4: now also IC3.17, IC3.18, R208.2; no longer IC5.17, IC5.18, R8.2
- net D5: now also IC3.15, IC3.16, R209.2; no longer IC5.15, IC5.16, R9.2
- net D6: now also IC3.13, IC3.14, R210.2; no longer IC5.13, IC5.14, R10.2
- net D7: now also IC3.11, IC3.12; no longer IC5.11, IC5.12
- net DATA_DIR: now also IC1.34, IC1.P$34, IC3.1; no longer IC5.1, U1.34, U1.P$34
- net DP: now also IC203.12, IC203.9; no longer IC3.12, IC3.9
- net GND: now also C1.1, C201.2, C204.2, C206.2, C207.2, C210.2, C8.2, IC1.13, IC1.18, IC1.23, IC1.28, IC1.3, IC1.33, IC1.38, IC1.8, IC1.P$13, IC1.P$18, IC1.P$23, IC1.P$28, IC1.P$3, IC1.P$33, IC1.P$38, IC1.P$8, IC201.10, IC201.7, IC201.8, IC201.9, IC202.10, IC202.14, IC202.7, IC203.10, IC203.14, IC203.7, IC3.19, IC5.5, IC5.6, IC5.7, IC5.8, IC5.9, IC6.3, J1.4, J2.A12, J2.B12, J2.MH1, J2.MH2, J2.MH3, J2.MH4, R3.2, R4.2, R5.2; no longer C1.2, C11.2, C12.2, C14.2, C15.2, C20.2, C8.1, IC1.10, IC1.14, IC1.7, IC3.14, IC3.7, IC6.10, IC6.7, IC6.8, IC6.9, IC7.10, IC7.19, IC7.5, IC7.6, IC7.7, IC7.8, IC7.9, IC8.3, J1.A12, J1.B12, J1.MH1, J1.MH2, J1.MH3, J1.MH4, R14.2, R17.2, R18.2, SV1.4, U1.13, U1.18, U1.23, U1.28, U1.3, U1.33, U1.38, U1.8, U1.P$13, U1.P$18, U1.P$23, U1.P$28, U1.P$3, U1.P$33, U1.P$38, U1.P$8
- net I/O: now also IC202.19, IC202.2; no longer IC1.19, IC1.2
- net IN_OE_CS: now also IC1.15, IC1.P$15, IC201.19, R6.2; no longer IC6.19, R37.2, U1.15, U1.P$15
- net KEYB_RX: now also IC1.20, IC1.P$20, IC5.17; no longer IC7.17, U1.20, U1.P$20
- net KEYB_TX: now also IC1.29, IC1.P$29, IC5.4; no longer IC7.4, U1.29, U1.P$29
- net KEYB_TX_ORIG: now also IC1.32, IC1.P$32, IC5.18; no longer IC7.18, U1.32, U1.P$32
- net MSG: now also IC202.12, IC202.9; no longer IC1.12, IC1.9
- net N$1: now also J2.B5, R4.1; no longer J1.B5, R14.1
- net N$12: now also R205.1; no longer R5.1
- net N$13: now also R206.1; no longer R6.1
- net N$14: now also R207.1; no longer R7.1
- net N$15: now also R208.1; no longer R8.1
- net N$18: now also R209.1; no longer R9.1
- net N$19: now also R210.1; no longer R10.1
- net N$2: now also J2.A5, R3.1; no longer J1.A5, R17.1
- net N$21: now also J1.2, RN1.6; no longer RN5.6, SV1.2
- net N$26: now also D1.C, IC1.39, IC1.P$39; no longer D2.C, U1.39, U1.P$39
- net N$3: now also IC6.2, R10.1; no longer IC8.2, R36.1
- net N$30: now also R223.1; no longer R4.1
- net N$4: now also IC6.1, R9.2; no longer IC8.1, R40.2
- net N$5: now also R223.2; no longer R4.2
- net N$6: now also R5.1; no longer R18.1
- net N$7: now also IC6.4; no longer IC8.4
- net OC_DRQ: now also D102.2; no longer D1.2
- net ODRQ: now also D102.1; no longer D1.1
- net OUT_LE1_DRQ: now also IC1.17, IC1.P$17, IC202.11, R8.2; no longer IC1.11, R39.2, U1.17, U1.P$17
- net OUT_LE2_RESET: now also IC1.19, IC1.P$19, IC203.11; no longer IC3.11, U1.19, U1.P$19
- net OUT_OE_INT: now also IC1.16, IC1.P$16, IC202.1, IC203.1, R7.2, R9.1; no longer IC1.1, IC3.1, R38.2, R40.1, U1.16, U1.P$16
- net REQ: now also IC203.19, IC203.2; no longer IC3.19, IC3.2
- net RST: now also IC201.3; no longer IC6.3
- net RST_C/D_REQ_NEOPIXEL: now also IC1.12, IC1.P$12, IC201.17, IC202.17, IC202.4, IC203.18, IC203.3, R10.2; no longer IC1.17, IC1.4, IC3.18, IC3.3, IC6.17, R36.2, U1.12, U1.P$12
- net SEL: now also IC201.2; no longer IC6.2
- net SEL_I/O_DP_A1: now also IC1.11, IC1.P$11, IC201.18, IC202.18, IC202.3, IC203.13, IC203.8; no longer IC1.18, IC1.3, IC3.13, IC3.8, IC6.18, U1.11, U1.P$11
- net VBUS: now also IC1.40, IC1.P$40; no longer U1.40, U1.P$40
- net VCC: now also C1.2, C201.1, C4.1, C5.1, IC201.1, IC201.20, IC5.1, IC5.20, R6.1, R7.1, R8.1; no longer C10.1, C12.1, C14.1, C8.2, IC6.1, IC6.20, IC7.1, IC7.20, R37.1, R38.1, R39.1
- net VCCBUS: now also C2.1, C3.1, IC3.20; no longer C1.1, C9.1, IC5.20
- net VCCIO: now also C204.1, C207.1, C210.1, IC202.20, IC203.20; no longer C2.1, C3.1, C5.1, IC1.20, IC3.20
- net ZKEYB_RX: now also J1.3, RN1.8; no longer RN5.8, SV1.3
- net ZKEYB_TX_ORIG: now also J1.1, RN1.5; no longer RN5.5, SV1.1
Routing:
- net GND: track 229.2 -> 232.0 mm

Commit message: fix for SCSI neopixel colors during start / run
Parts:
- removed R9: 220R, rcl:R0603
- added C11: 100 nF, rcl:C0603
- added IC207: 74AHCT1G08GW,125, 74AHCT1G08GW_125:SOT65P212X110-5N
- added R109: 10k, rcl:R0603
Connections:
- net 5V: now also C11.1, IC207.5, R109.1
- net GND: now also C11.2, IC207.3
- net N$4: now also IC207.4, R109.2; no longer R9.2
- net OUT_LE1_DRQ: now also IC207.2
- net OUT_LE2_RESET: now also IC207.1
- net OUT_OE_INT: no longer R9.1
Routing:
- net 5V: track 214.5 -> 232.6 mm
- net OUT_LE1_DRQ: track 71.9 -> 82.5 mm, vias 3 -> 5
- net N$4: track 4.77 -> 14.0 mm, vias 0 -> 2
- net OUT_LE2_RESET: track 71.0 -> 79.4 mm, vias 2 -> 4
- net GND: track 232.0 -> 237.2 mm, vias 67 -> 68
- net OUT_OE_INT: track 107.2 -> 102.7 mm
- net KEYB_RX: track 35.6 -> 36.1 mm

Commit message: hdd pcb has now different led connections for scsi and for acsi
Parts:
- removed C11: 100 nF, rcl:C0603
- removed IC207: 74AHCT1G08GW,125, 74AHCT1G08GW_125:SOT65P212X110-5N
- removed R10: 220R, rcl:R0603
- removed R109: 10k, rcl:R0603
- added R150, R250, R251: 220R, rcl:R0603
- added R151: 10k, rcl:R0603
- moved LED1 48.0 mm to (-26.1, 38.4)
- moved R5 47.6 mm to (-26.1, 35.8)
- moved C10 7.35 mm to (2.30, 76.4), turned to 90 degrees
- moved R203 4.01 mm to (15.3, 29.2)
- moved R202 0.96 mm to (14.4, 31.4), turned to 270 degrees
Connections:
- removed net RST_C/D_REQ_NEOPIXEL: IC1.12, IC1.P$12, IC201.17, IC202.17, IC202.4, IC203.18, IC203.3, R10.2
- new net RST_C/D_REQ: IC1.12, IC1.P$12, IC201.17, IC202.17, IC202.4, IC203.18, IC203.3, R150.2
- net 5V: now also R151.2; no longer C11.1, IC207.5, R109.1
- net GND: no longer C11.2, IC207.3
- net N$3: now also R150.1, R250.1; no longer R10.1
- net N$4: now also R151.1, R251.1; no longer IC207.4, R109.2
- net OUT_LE1_DRQ: now also R250.2; no longer IC207.2
- net OUT_LE2_RESET: now also R251.2; no longer IC207.1
Routing:
- net RST_C/D_REQ: track 0.00 -> 98.8 mm, vias 0 -> 4
- net RST_C/D_REQ_NEOPIXEL: track 98.8 -> 0.00 mm, vias 4 -> 0
- net OUT_OE_INT: track 102.7 -> 85.7 mm, vias 4 -> 3
- net OUT_LE2_RESET: track 79.4 -> 93.7 mm
- net GND: track 237.2 -> 228.4 mm
- net N$4: track 14.0 -> 6.25 mm, vias 2 -> 0
- net 5V: track 232.6 -> 228.8 mm, vias 8 -> 10
- net OUT_LE1_DRQ: track 82.5 -> 84.2 mm
- net TP_ON: track 102.6 -> 101.0 mm
- net N$3: track 8.71 -> 10.3 mm
- net ATN_MSG: track 60.9 -> 59.7 mm
- net N$8: track 2.23 -> 3.35 mm
- net 5V_IN: track 45.1 -> 44.3 mm
- net KEYB_TX_ORIG: track 35.8 -> 35.1 mm
Other:
- board text added: "A"
- board text added: "Cosmo2ex HDD 4.05"
- board text added: "PRESENT"
- board text added: "S"
- board text added: "TRMPWR"
- board text removed: "Cosmo2ex HDD 4.04"
- board text removed: "INSTALLED"
- board text removed: "SCSI"
