File: devices/v40_pico_hdd/ce_hdd_v40.sch (EAGLE design)
At the start: 108 parts, among them IC1 74LVC373APW,118, IC11 TLV1117LV33DCYR, IC12 74LVC245AT20-13, IC2 74LVC245AT20-13, IC3 74LVC373APW,118, IC4 SN74AHCT1G125DBVR, IC5 74LVC245AT20-13, IC6 74LVC245AT20-13, IC7 74LVC245AT20-13, IC9 AZ1117H-ADJTRE1, J1 USB4125-GF-A, Q1 FDV304P, Q10 FDV304P, Q11 FDV304P, Q12 FDV304P, Q13 FDV304P, Q14 FDV304P, Q15 FDV304P, Q16 FDV304P, Q17 FDV304P, Q18 FDV304P, Q2 FDV304P, Q3 FDV304P, Q4 FDV304P, Q5 FDV304P, Q6 FDV304P, Q7 FDV304P, Q8 FDV304P, Q9 FDV304P, U1 RASPBERRY_PICOSMD-TH

Commit message: first version of merged hdd routed
Parts:
- removed C16, C17, C19: 100 nF, rcl:C-EUC0603
- added LED3: WS2812C-2020, WS2812C-2020:WS2812C-2020
- C18: device rcl:C-EUC0805 -> rcl:C-EUC0603
- U$1: value RSSM1011C3BK -> SMSR-1; device RSSM1011C3BK:RSSM1011C3BK -> ce_fdd_v40:SMSR-1
Connections:
- net 5V: now also LED3.VDD
- net GND: now also LED3.GND; no longer C16.2, C17.2, C19.2
- net N$7: now also LED3.DI
- net VCC: no longer C16.1, C17.1, C19.1
- net VCCBUS: now also C1.1, C9.1
- net VCCIO: no longer C1.1, C9.1
Other:
- moved on the sheet: C18

Commit message: routing finished, few tweaks done
Parts:
- removed D3: TS4148_RBG, TS4148_RBG:TS4148_RBG
- removed IC4: SN74AHCT1G125DBVR, SN74AHCT1G125DBVR:SN74AHCT1G125DBVR
- added D4: BAT54WSTR, BAT54WSTR:BAT54WSTR
- added IC8: 74AHCT1G08GW,125, 74AHCT1G08GW_125:74AHCT1G08GW,125
- added R37, R38, R39: 10k, rcl:R-EU_R0603
- added R40: 220R, rcl:R-EU_R0603
- D1: value TS4148_RBG -> BAT54WSTR; device TS4148_RBG:TS4148_RBG -> BAT54WSTR:BAT54WSTR; DESCRIPTION Diodes - General Purpose, Power, Switching 75V, 0.15A, Swit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 -> DIODE SCHOTTKY 30V 200MA SOD323; HEIGHT 0.85mm -> 1mm; MANUFACTURER_NAME Taiwan Semiconductor -> SMC Diode Solutions; MANUFACTURER_PART_NUMBER TS4148 RBG -> BAT54WSTR
Connections:
- new net N$4: IC8.B, R40.2
- net 5V: now also IC8.VCC; no longer IC4.VCC
- net GND: now also IC8.GND; no longer IC4.!OE, IC4.GND
- net IN_OE_CS: now also R37.2
- net N$3: now also IC8.A; no longer IC4.A
- net N$7: now also IC8.Y; no longer IC4.Y
- net OC_INT: now also D4.A; no longer D3.A
- net OINT: now also D4.K; no longer D3.K
- net OUT_LE1_DRQ: now also R39.2
- net OUT_OE_INT: now also R38.2, R40.1
- net VCC: now also R37.1, R38.1, R39.1
Changed lines of the file:
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@@
 <part name="R31" library="rcl" deviceset="R-EU_" device="R0603" value="10k"/>
 <part name="R29" library="rcl" deviceset="R-EU_" device="R0603" value="10k"/>
-<part name="D3" library="TS4148_RBG" deviceset="TS4148_RBG" device=""/>
-<part name="D1" library="TS4148_RBG" deviceset="TS4148_RBG" device="">
-<attribute name="DESCRIPTION" value="Diodes - General Purpose, Power, Switching 75V, 0.15A, Switching Diode &amp; Array"/>
-<attribute name="HEIGHT" value="0.85mm"/>
-<attribute name="MANUFACTURER_NAME" value="Taiwan Semiconductor"/>
-<attribute name="MANUFACTURER_PART_NUMBER" value="TS4148 RBG"/>
-<attribute name="TME_ELECTRONIC_COMPONENTS_PART_NUMBER" value=""/>
-<attribute name="TME_ELECTRONIC_COMPONENTS_PRICE-STOCK" value=""/>
-</part>
 <part name="GND30" library="supply1" deviceset="GND" device=""/>
 <part name="IC12" library="74LVC245AT20-13" deviceset="74LVC245AT20-13" device=""/>
@@
 <part name="R35" library="rcl" deviceset="R-EU_" device="R0603" value="0R"/>
 <part name="LED2" library="WS2812C-2020" deviceset="WS2812C-2020" device=""/>
-<part name="IC4" library="SN74AHCT1G125DBVR" deviceset="SN74AHCT1G125DBVR" device=""/>
 <part name="GND6" library="supply1" deviceset="GND" device=""/>
 <part name="C20" library="rcl" deviceset="C-EU" device="C0603" value="100 nF"/>
@@
 <attribute name="TME_ELECTRONIC_COMPONENTS_PRICE-STOCK" value=""/>
 </part>
+<part name="R37" library="rcl" deviceset="R-EU_" device="R0603" value="10k"/>
+<part name="R38" library="rcl" deviceset="R-EU_" device="R0603" value="10k"/>
+<part name="R39" library="rcl" deviceset="R-EU_" device="R0603" value="10k"/>
+<part name="IC8" library="74AHCT1G08GW_125" deviceset="74AHCT1G08GW,125" device=""/>
+<part name="R40" library="rcl" deviceset="R-EU_" device="R0603" value="220R"/>
+<part name="D4" library="BAT54WSTR" deviceset="BAT54WSTR" device=""/>
+<part name="D1" library="BAT54WSTR" deviceset="BAT54WSTR" device="">
+<attribute name="DESCRIPTION" value="DIODE SCHOTTKY 30V 200MA SOD323"/>
+<attribute name="HEIGHT" value="1mm"/>
+<attribute name="MANUFACTURER_NAME" value="SMC Diode Solutions"/>
+<attribute name="MANUFACTURER_PART_NUMBER" value="BAT54WSTR"/>
+<attribute name="TME_ELECTRONIC_COMPONENTS_PART_NUMBER" value=""/>
+<attribute name="TME_ELECTRONIC_COMPONENTS_PRICE-STOCK" value=""/>
+</part>
 </parts>
 <sheets>
@@
 <instance part="R31" gate="G$1" x="106.68" y="205.74" smashed="yes" rot="MR180"/>
 <instance part="R29" gate="G$1" x="106.68" y="210.82" smashed="yes" rot="MR180"/>
-<instance part="D3" gate="G$1" x="238.76" y="109.22"/>
-<instance part="D1" gate="G$1" x="238.76" y="99.06"/>
 <instance part="GND30" gate="1" x="198.12" y="96.52" smashed="yes">
 <attribute name="VALUE" x="195.58" y="93.98" size="1.778" layer="96"/>
@@
 <instance part="RN3" gate="G$1" x="43.18" y="144.78" rot="R180"/>
 <instance part="RN4" gate="G$1" x="43.18" y="127" rot="R180"/>
+<instance part="D4" gate="G$1" x="238.76" y="109.22"/>
+<instance part="D1" gate="G$1" x="238.76" y="99.06"/>
 </instances>
 <busses>
@@
 <wire x1="254" y1="109.22" x2="259.08" y2="109.22" width="0.1524" layer="91"/>
 <label x="254.762" y="107.95" size="0.8128" layer="95" font="vector"/>
-<pinref part="D3" gate="G$1" pin="A"/>
+<pinref part="D4" gate="G$1" pin="A"/>
 </segment>
 <segment>
@@
 <label x="229.87" y="106.934" size="1.016" layer="95" font="vector"/>
 <wire x1="233.68" y1="106.68" x2="233.68" y2="99.06" width="0.1524" layer="91"/>
-<pinref part="D1" gate="G$1" pin="K"/>
 <wire x1="233.68" y1="99.06" x2="238.76" y2="99.06" width="0.1524" layer="91"/>
+<pinref part="D1" gate="G$1" pin="K"/>
 </segment>
 </net>
@@
 <wire x1="226.06" y1="109.22" x2="238.76" y2="109.22" width="0.1524" layer="91"/>
 <label x="229.87" y="109.474" size="1.016" layer="95" font="vector"/>
-<pinref part="D3" gate="G$1" pin="K"/>
+<pinref part="D4" gate="G$1" pin="K"/>
 </segment>
 </net>
@@
 <instance part="GND10" gate="1" x="281.94" y="137.16"/>
 <instance part="LED2" gate="G$1" x="203.2" y="48.26" rot="R270"/>
-<instance part="IC4" gate="G$1" x="142.24" y="45.72"/>
 <instance part="GND6" gate="1" x="139.7" y="35.56"/>
 <instance part="C20" gate="G$1" x="172.72" y="35.56" smashed="yes">
@@
 <instance part="U$1" gate="G$1" x="259.08" y="170.18"/>
 <instance part="LED3" gate="G$1" x="223.52" y="48.26" rot="R270"/>
+<instance part="R37" gate="G$1" x="-30.48" y="137.16" smashed="yes">
+<attribute name="VALUE" x="-37.592" y="137.668" size="1.778" layer="96"/>
+</instance>
+<instance part="R38" gate="G$1" x="-30.48" y="134.62" smashed="yes">
+<attribute name="VALUE" x="-37.592" y="135.128" size="1.778" layer="96"/>
+</instance>
+<instance part="R39" gate="G$1" x="-30.48" y="132.08" smashed="yes">
+<attribute name="VALUE" x="-37.592" y="130.048" size="1.778" layer="96"/>
+</instance>
+<instance part="IC8" gate="G$1" x="142.24" y="45.72"/>
+<instance part="R40" gate="G$1" x="132.08" y="45.72" smashed="yes" rot="MR180">
+<attribute name="VALUE" x="129.54" y="48.768" size="1.778" layer="96" rot="MR180"/>
+</instance>
 </instances>
 <busses>
@@
 <label x="75.184" y="165.608" size="0.8128" layer="95" font="vector"/>
 </segment>
+<segment>
+<pinref part="R37" gate="G$1" pin="1"/>
+<wire x1="-35.56" y1="137.16" x2="-38.1" y2="137.16" width="0.1524" layer="91"/>
+<wire x1="-38.1" y1="137.16" x2="-38.1" y2="134.62" width="0.1524" layer="91"/>
+<pinref part="R39" gate="G$1" pin="1"/>
+<wire x1="-38.1" y1="134.62" x2="-38.1" y2="132.08" width="0.1524" layer="91"/>
+<wire x1="-38.1" y1="132.08" x2="-35.56" y2="132.08" width="0.1524" layer="91"/>
+<pinref part="R38" gate="G$1" pin="1"/>
+<wire x1="-35.56" y1="134.62" x2="-38.1" y2="134.62" width="0.1524" layer="91"/>
+<junction x="-38.1" y="134.62"/>
+<wire x1="-38.1" y1="134.62" x2="-43.18" y2="134.62" width="0.1524" layer="91"/>
+<label x="-43.18" y="135.128" size="0.8128" layer="95" font="vector"/>
+</segment>
 </net>
 <net name="GND" class="0">
@@
 </segment>
 <segment>
-<pinref part="IC4" gate="G$1" pin="!OE"/>
-<wire x1="142.24" y1="45.72" x2="139.7" y2="45.72" width="0.1524" layer="91"/>
-<wire x1="139.7" y1="45.72" x2="139.7" y2="40.64" width="0.1524" layer="91"/>
-<pinref part="IC4" gate="G$1" pin="GND"/>
 <wire x1="139.7" y1="40.64" x2="139.7" y2="38.1" width="0.1524" layer="91"/>
 <wire x1="142.24" y1="40.64" x2="139.7" y2="40.64" width="0.1524" layer="91"/>
-<junction x="139.7" y="40.64"/>
 <pinref part="GND6" gate="1" pin="GND"/>
+<pinref part="IC8" gate="G$1" pin="GND"/>
 </segment>
 <segment>
@@
 <wire x1="200.66" y1="58.42" x2="180.34" y2="58.42" width="0.1524" layer="91"/>
 <junction x="180.34" y="58.42"/>
-<pinref part="IC4" gate="G$1" pin="VCC"/>
 <wire x1="167.64" y1="43.18" x2="172.72" y2="43.18" width="0.1524" layer="91"/>
 <junction x="180.34" y="43.18"/>
@@
 <wire x1="220.98" y1="58.42" x2="220.98" y2="48.26" width="0.1524" layer="91"/>
 <junction x="200.66" y="58.42"/>
+<pinref part="IC8" gate="G$1" pin="VCC"/>
 </segment>
 </net>
@@
 <segment>
 <pinref part="R36" gate="G$1" pin="2"/>
-<wire x1="127" y1="43.18" x2="111.252" y2="43.18" width="0.1524" layer="91"/>
-<label x="111.506" y="43.434" size="0.8128" layer="95" font="vector"/>
+<wire x1="127" y1="43.18" x2="111.76" y2="43.18" width="0.1524" layer="91"/>
+<label x="111.76" y="43.434" size="0.8128" layer="95" font="vector"/>
 </segment>
 </net>
@@
 <segment>
 <pinref part="U1" gate="U$1" pin="GP11"/>
-<wire x1="-7.62" y1="137.16" x2="-17.78" y2="137.16" width="0.1524" layer="91"/>
+<wire x1="-7.62" y1="137.16" x2="-25.4" y2="137.16" width="0.1524" layer="91"/>
 <label x="-17.78" y="137.414" size="0.8128" layer="95" font="vector"/>
+<pinref part="R37" gate="G$1" pin="2"/>
 </segment>
 </net>
@@
 <segment>
 <pinref part="U1" gate="U$1" pin="GP13"/>
-<wire x1="-7.62" y1="132.08" x2="-17.78" y2="132.08" width="0.1524" layer="91"/>
+<wire x1="-7.62" y1="132.08" x2="-25.4" y2="132.08" width="0.1524" layer="91"/>
 <label x="-17.78" y="132.334" size="0.8128" layer="95" font="vector"/>
+<pinref part="R39" gate="G$1" pin="2"/>
 </segment>
 </net>
@@
 <segment>
 <pinref part="U1" gate="U$1" pin="GP12"/>
-<wire x1="-7.62" y1="134.62" x2="-17.78" y2="134.62" width="0.1524" layer="91"/>
+<wire x1="-7.62" y1="134.62" x2="-25.4" y2="134.62" width="0.1524" layer="91"/>
 <label x="-17.78" y="134.874" size="0.8128" layer="95" font="vector"/>
+<pinref part="R38" gate="G$1" pin="2"/>
+</segment>
+<segment>
+<pinref part="R40" gate="G$1" pin="1"/>
+<wire x1="127" y1="45.72" x2="111.76" y2="45.72" width="0.1524" layer="91"/>
+<label x="111.76" y="45.974" size="0.8128" layer="95" font="vector"/>
 </segment>
 </net>
@@
 <net name="N$7" class="0">
 <segment>
-<pinref part="IC4" gate="G$1" pin="Y"/>
 <pinref part="LED2" gate="G$1" pin="DI"/>
 <wire x1="167.64" y1="45.72" x2="193.04" y2="45.72" width="0.1524" layer="91"/>
@@
 <wire x1="223.52" y1="50.8" x2="223.52" y2="48.26" width="0.1524" layer="91"/>
 <junction x="203.2" y="50.8"/>
+<pinref part="IC8" gate="G$1" pin="Y"/>
 </segment>
 </net>
@@
 <segment>
 <pinref part="R36" gate="G$1" pin="1"/>
-<pinref part="IC4" gate="G$1" pin="A"/>
 <wire x1="137.16" y1="43.18" x2="142.24" y2="43.18" width="0.1524" layer="91"/>
+<pinref part="IC8" gate="G$1" pin="A"/>
+</segment>
+</net>
+<net name="N$4" class="0">
+<segment>
+<pinref part="IC8" gate="G$1" pin="B"/>
+<pinref part="R40" gate="G$1" pin="2"/>
+<wire x1="142.24" y1="45.72" x2="137.16" y2="45.72" width="0.1524" layer="91"/>
 </segment>
 </net>

Commit message: minor components adjustment
Parts:
- C14, C15, C2, C24, C30: device rcl:C-EUC0805 -> rcl:C-EUC0603
- R18: value 470R -> 10k

Commit message: components renamed, components renumbered, ACSI and SCSI variants created
Parts:
- removed C11, C12, C13, C20, C23: 100 nF, rcl:C-EUC0603
- removed C14, C15, C18, C30: 1 uF, rcl:C-EUC0603
- removed D2: SK110-DIO, diode:DIODE-DO214AC
- removed D4: BAT54WSTR, BAT54WSTR:BAT54WSTR
- removed IC11: TLV1117LV33DCYR, TLV1117LV33DCYR:TLV1117LV33DCYR
- removed IC12, IC7: 74LVC245AT20-13, 74LVC245AT20-13:74LVC245AT20-13
- removed IC8: 74AHCT1G08GW,125, 74AHCT1G08GW_125:74AHCT1G08GW,125
- removed JP1: (no value), jumper:JP1E
- removed Q1, Q10, Q11, Q12, Q13, Q14, Q15, Q16, Q17, Q18, Q2, Q3, Q4, Q5, Q6, Q7, Q8, Q9: FDV304P, IRLML6401TRPBF:IRLML6401TRPBF
- removed R11, R13, R16, R19, R22, R23, R24, R25, R26, R27, R28: 110 R, rcl:R-EU_R0603
- removed R14, R17: 5k1 (1%), rcl:R-EU_R0603
- removed R18, R29, R30, R31, R32, R37, R38, R39: 10k, rcl:R-EU_R0603
- removed R33, R36, R40: 220R, rcl:R-EU_R0603
- removed R34, R35: 0R, rcl:R-EU_R0603
- removed RN2, RN3, RN4, RN5: DR1206-47R-4/8, resistor-net:CTS742C083
- removed SV1: (no value), con-lstb:MA04-1
- removed U$1: SMSR-1, ce_fdd_v40:SMSR-1
- removed U$3: M19, con_subd19:M19
- removed U1: RASPBERRY_PICOSMD-TH, RpiPico:RASPBERRY_PICOSMD-TH
- added C101, C203, C210: 1 uF, rcl:C-EUC0603
- added C201, C202, C204, C205: 100 nF, rcl:C-EUC0603
- added C206, C207: 10 uF, 293D106X9016B2TE3:293D106X9016B2TE3
- added D101, D102: BAT54WSTR, BAT54WSTR:BAT54WSTR
- added IC101, IC201: 74LVC245AT20-13, 74LVC245AT20-13:74LVC245AT20-13
- added IC202, IC203: 74LVC373APW,118, 74LVC373APW_118:74LVC373APW,118
- added IC4: TLV1117LV33DCYR, TLV1117LV33DCYR:TLV1117LV33DCYR
- added J101: M19, con_subd19:M19
- added J2: USB4125-GF-A, USB4125-GF-A:USB4125-GF-A
- added JP201: (no value), jumper:JP1E
- added Q201, Q202, Q203, Q204, Q205, Q206, Q207, Q208, Q209, Q210, Q211, Q212, Q213, Q214, Q215, Q216, Q217, Q218: FDV304P, IRLML6401TRPBF:IRLML6401TRPBF
- added R101, R201: 0R, rcl:R-EU_R0603
- added R102, R103, R104, R202: 10k, rcl:R-EU_R0603
- added R203: 220R, rcl:R-EU_R0603
- added R204, R205, R206, R207, R208, R209, R210, R211, R212, R213, R214, R215, R216, R217, R218, R219, R220, R221: 110 R, rcl:R-EU_R0603
- added R223: 150 R, rcl:R-EU_R0603
- added RN101, RN102, RN103, RN104: DR1206-47R-4/8, resistor-net:CTS742C083
- added SW1: SMSR-1, ce_fdd_v40:SMSR-1
- C10, C5: value 10 uF -> 100 nF; device 293D106X9016B2TE3:293D106X9016B2TE3 -> rcl:C-EUC0603; DESCRIPTION Solid Tantalum Surface Mount Chip Capacitors TANTAMOUNT(TM)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 -> (none); HEIGHT 2.1mm -> (none); MANUFACTURER_NAME Vishay -> (none); MANUFACTURER_PART_NUMBER 293D106X9016B2TE3 -> (none)
- C2: value 1 uF -> 100 nF
- C6, C8: value 100 nF -> 1 uF
- D1: value BAT54WSTR -> SK110-DIO; device BAT54WSTR:BAT54WSTR -> diode:DIODE-DO214AC; DESCRIPTION DIODE SCHOTTKY 30V 200MA SOD323 -> (none); HEIGHT 1mm -> (none); MANUFACTURER_NAME SMC Diode Solutions -> (none); MANUFACTURER_PART_NUMBER BAT54WSTR -> (none)
- IC1: value 74LVC373APW,118 -> RASPBERRY_PICOSMD-TH; device 74LVC373APW_118:74LVC373APW,118 -> RpiPico:RASPBERRY_PICOSMD-TH
- IC3: value 74LVC373APW,118 -> 74LVC245AT20-13; device 74LVC373APW_118:74LVC373APW,118 -> 74LVC245AT20-13:74LVC245AT20-13
- IC6: value 74LVC245AT20-13 -> 74AHCT1G08GW,125; device 74LVC245AT20-13:74LVC245AT20-13 -> 74AHCT1G08GW_125:74AHCT1G08GW,125
- J1: value USB4125-GF-A -> (none); device USB4125-GF-A:USB4125-GF-A -> con-lstb:MA04-1
- R1, R6, R7, R8: value 110 R -> 10k
- R10, R9: value 110 R -> 220R
- R3: value 10k -> 5k1 (1%)
- R4: value 150 R -> 5k1 (1%)
- R5: value 110 R -> 1k
- renumbered C21 to C208, C22 to C209, C24 to C211, IC9 to IC204, R12 to R224, R15 to R222, R20 to R125, R21 to R225, SV2 to J203, U$2 to J201, X1 to J202
Connections:
- net 5V: now also C10.1, C206.+, C8.1, C9.1, D1.A, IC4.INPUT, IC6.VCC, R1.2, SW1.P$2; no longer C11.1, C15.1, C20.1, C4.+, D2.A, IC11.INPUT, IC8.VCC, R3.2, U$1.P$2
- net 5V_IN: now also J2.VBUS_1, J2.VBUS_2, SW1.P$1; no longer J1.VBUS_1, J1.VBUS_2, U$1.P$1
- net AA1: now also J101.16, RN103.4; no longer RN3.4, U$3.16
- net AAAA: now also Q201.D, R204.1; no longer Q1.D, R1.1
- net AACK: now also J101.14, RN102.3; no longer RN2.3, U$3.14
- net ACK: now also IC203.D1, IC203.D6, R215.2; no longer IC3.D1, IC3.D6, R22.2
- net ACS: now also J101.9, RN104.4; no longer RN4.4, U$3.9
- net AD0: now also J101.1, RN101.4; no longer RN1.4, U$3.1
- net AD1: now also J101.2, RN101.3; no longer RN1.3, U$3.2
- net AD2: now also J101.3, RN101.1; no longer RN1.1, U$3.3
- net AD3: now also J101.4, RN102.4; no longer RN2.4, U$3.4
- net AD4: now also J101.5, RN102.2; no longer RN2.2, U$3.5
- net AD5: now also J101.6, RN102.1; no longer RN2.1, U$3.6
- net AD6: now also J101.7, RN103.3; no longer RN3.3, U$3.7
- net AD7: now also J101.8, RN103.2; no longer RN3.2, U$3.8
- net ADRQ: now also J101.19, RN104.3; no longer RN4.3, U$3.19
- net AINT: now also J101.10, RN104.2; no longer RN4.2, U$3.10
- net ARESET: now also J101.12, RN101.2; no longer RN1.2, U$3.12
- net ARNW: now also J101.18, RN103.1; no longer RN3.1, U$3.18
- net ATN: now also IC201.A5, R213.2; no longer IC6.A5, R16.2
- net ATN_MSG: now also IC1.GP26, IC201.B5, IC202.D3, IC202.D4; no longer IC1.D3, IC1.D4, IC6.B5, U1.GP26
- net BA1: now also IC101.A2, RN103.5; no longer IC12.A2, RN3.5
- net BACK: now also IC101.A3, R103.2, RN102.6; no longer IC12.A3, R31.2, RN2.6
- net BCS: now also IC101.A1, R102.2, RN104.5; no longer IC12.A1, R29.2, RN4.5
- net BRESET: now also IC101.A4, R104.2, RN101.7; no longer IC12.A4, R30.2, RN1.7
- net BSY: now also IC201.A4, IC202.Q2, IC202.Q5, R214.2; no longer IC1.Q2, IC1.Q5, IC6.A4, R19.2
- net BSY_IN: now also IC201.B4; no longer IC6.B4
- net C/D: now also IC202.Q1, IC202.Q6, R219.2; no longer IC1.Q1, IC1.Q6, R26.2
- net C0: now also IC1.GP0; no longer U1.GP0
- net C1: now also IC1.GP1; no longer U1.GP1
- net C2: now also IC1.GP2; no longer U1.GP2
- net C3: now also IC1.GP3; no longer U1.GP3
- net C4: now also IC1.GP4, IC3.A1, IC3.A2; no longer IC5.A1, IC5.A2, U1.GP4
- net C5: now also IC1.GP5, IC3.A3, IC3.A4; no longer IC5.A3, IC5.A4, U1.GP5
- net C6: now also IC1.GP6, IC3.A5, IC3.A6; no longer IC5.A5, IC5.A6, U1.GP6
- net C7: now also IC1.GP7, IC3.A7, IC3.A8; no longer IC5.A7, IC5.A8, U1.GP7
- net CACK: now also IC1.GP10, IC101.B3, IC203.Q1, IC203.Q6; no longer IC12.B3, IC3.Q1, IC3.Q6, U1.GP10
- net CKEYB_RX: now also IC5.A2, R2.1, RN1.1; no longer IC7.A2, R3.1, RN5.1
- net CKEYB_TX: now also IC5.B3, RN1.3; no longer IC7.B3, RN5.3
- net CKEYB_TX_ORIG: now also IC5.A1, R1.1, RN1.4; no longer IC7.A1, R2.1, RN5.4
- net D0: now also R204.2, RN101.5; no longer R1.2, RN1.5
- net D1: now also R205.2, RN101.6; no longer R5.2, RN1.6
- net D2: now also R206.2, RN101.8; no longer R6.2, RN1.8
- net D3: now also R207.2, RN102.5; no longer R7.2, RN2.5
- net D4: now also IC3.B1, IC3.B2, R208.2, RN102.7; no longer IC5.B1, IC5.B2, R8.2, RN2.7
- net D5: now also IC3.B3, IC3.B4, R209.2, RN102.8; no longer IC5.B3, IC5.B4, R9.2, RN2.8
- net D6: now also IC3.B5, IC3.B6, R210.2, RN103.6; no longer IC5.B5, IC5.B6, R10.2, RN3.6
- net D7: now also IC3.B7, IC3.B8, R211.2, RN103.7; no longer IC5.B7, IC5.B8, R11.2, RN3.7
- net DATA_DIR: now also IC1.GP28, IC3.DIR; no longer IC5.DIR, U1.GP28
- net DP: now also IC203.Q3, IC203.Q4, R212.2; no longer IC3.Q3, IC3.Q4, R13.2
- net GND: now also C1.1, C10.2, C101.2, C201.2, C202.2, C203.2, C204.2, C205.2, C206.-, C207.-, C210.2, C5.2, C8.2, IC101.!OE, IC101.A7, IC101.A8, IC101.GND, IC201.A6, IC201.A7, IC201.A8, IC201.GND, IC202.D2, IC202.D5, IC202.GND, IC203.D2, IC203.D5, IC203.GND, IC3.!OE, IC4.GND, IC5.A4, IC5.A5, IC5.A6, IC5.A7, IC5.A8, J1.4, J101.11, J101.13, J101.15, J101.17, J2.GND_1, J2.GND_2, J2.MH1, J2.MH2, J2.MH3, J2.MH4, JP201.2, R104.1, R3.2, R4.2, R5.2; no longer C1.2, C10.-, C11.2, C12.2, C13.2, C14.2, C15.2, C18.2, C20.2, C23.2, C30.2, C5.-, C8.1, IC1.D2, IC1.D5, IC11.GND, IC12.!OE, IC12.A7, IC12.A8, IC12.GND, IC3.D2, IC3.D5, IC6.A6, IC6.A7, IC6.A8, IC7.!OE, IC7.A4, IC7.A5, IC7.A6, IC7.A7, IC7.A8, IC7.GND, IC8.GND, J1.GND_1, J1.GND_2, J1.MH1, J1.MH2, J1.MH3, J1.MH4, JP1.2, R14.2, R17.2, R18.2, R30.1, SV1.4, U$3.11, U$3.13, U$3.15, U$3.17, U1.GND
- net I/O: now also IC202.Q0, IC202.Q7, R221.2; no longer IC1.Q0, IC1.Q7, R28.2
- net IN_OE_CS: now also IC1.GP11, IC101.B1, IC201.!OE, R6.2; no longer IC12.B1, IC6.!OE, R37.2, U1.GP11
- net KEYB_RX: now also IC1.GP15, IC5.B2; no longer IC7.B2, U1.GP15
- net KEYB_TX: now also IC1.GP22, IC5.A3; no longer IC7.A3, U1.GP22
- net KEYB_TX_ORIG: now also IC1.GP27, IC5.B1; no longer IC7.B1, U1.GP27
- net MSG: now also IC202.Q3, IC202.Q4, R217.2; no longer IC1.Q3, IC1.Q4, R24.2
- net N$1: now also J2.CC2, R4.1; no longer J1.CC2, R14.1
- net N$100: now also Q211.D, R214.1; no longer Q11.D, R19.1
- net N$101: now also Q212.D, R215.1; no longer Q12.D, R22.1
- net N$102: now also Q213.D, R216.1; no longer Q13.D, R23.1
- net N$103: now also Q214.D, R217.1; no longer Q14.D, R24.1
- net N$104: now also Q215.D, R218.1; no longer Q15.D, R25.1
- net N$105: now also Q216.D, R219.1; no longer Q16.D, R26.1
- net N$106: now also Q217.D, R220.1; no longer Q17.D, R27.1
- net N$107: now also Q218.D, R221.1; no longer Q18.D, R28.1
- net N$12: now also Q202.D, R205.1; no longer Q2.D, R5.1
- net N$13: now also Q203.D, R206.1; no longer Q3.D, R6.1
- net N$14: now also Q204.D, R207.1; no longer Q4.D, R7.1
- net N$15: now also Q205.D, R208.1; no longer Q5.D, R8.1
- net N$18: now also Q206.D, R209.1; no longer Q6.D, R9.1
- net N$19: now also Q207.D, R210.1; no longer Q7.D, R10.1
- net N$2: now also J2.CC1, R3.1; no longer J1.CC1, R17.1
- net N$20: now also Q208.D, R211.1; no longer Q8.D, R11.1
- net N$21: now also J1.2, RN1.6; no longer RN5.6, SV1.2
- net N$22: now also Q209.D, R212.1; no longer Q9.D, R13.1
- net N$24: now also Q210.D, R213.1; no longer Q10.D, R16.1
- net N$26: now also D1.C, IC1.VSYS; no longer D2.C, U1.VSYS
- net N$3: now also IC6.A, R10.1; no longer IC8.A, R36.1
- net N$30: now also R223.1; no longer R4.1
- net N$4: now also IC6.B, R9.2; no longer IC8.B, R40.2
- net N$5: now also R223.2; no longer R4.2
- net N$6: now also R5.1; no longer R18.1
- net N$7: now also IC6.Y; no longer IC8.Y
- net N$8: now also JP201.1, R203.2; no longer JP1.1, R33.2
- net OC_DRQ: now also D102.A, RN104.6; no longer D1.A, RN4.6
- net OC_INT: now also D101.A, RN104.7; no longer D4.A, RN4.7
- net ODRQ: now also D102.K, IC101.B6; no longer D1.K, IC12.B6
- net OINT: now also D101.K, IC101.B5; no longer D4.K, IC12.B5
- net OUT_LE1_DRQ: now also IC1.GP13, IC101.A6, IC202.LE, R8.2; no longer IC1.LE, IC12.A6, R39.2, U1.GP13
- net OUT_LE2_RESET: now also IC1.GP14, IC101.B4, IC203.LE; no longer IC12.B4, IC3.LE, U1.GP14
- net OUT_OE_INT: now also IC1.GP12, IC101.A5, IC202.!OE, IC203.!OE, R7.2, R9.1; no longer IC1.!OE, IC12.A5, IC3.!OE, R38.2, R40.1, U1.GP12
- net REQ: now also IC203.Q0, IC203.Q7, R220.2; no longer IC3.Q0, IC3.Q7, R27.2
- net RST: now also IC201.A2, R216.2; no longer IC6.A2, R23.2
- net RST_C/D_REQ_NEOPIXEL: now also IC1.GP9, IC201.B2, IC202.D1, IC202.D6, IC203.D0, IC203.D7, R10.2; no longer IC1.D1, IC1.D6, IC3.D0, IC3.D7, IC6.B2, R36.2, U1.GP9
- net SEL: now also IC201.A1, R218.2; no longer IC6.A1, R25.2
- net SEL_I/O_DP_A1: now also IC1.GP8, IC101.B2, IC201.B1, IC202.D0, IC202.D7, IC203.D3, IC203.D4; no longer IC1.D0, IC1.D7, IC12.B2, IC3.D3, IC3.D4, IC6.B1, U1.GP8
- net TP_ON: now also Q201.G, Q202.G, Q203.G, Q204.G, Q205.G, Q206.G, Q207.G, Q208.G, Q209.G, Q210.G, Q211.G, Q212.G, Q213.G, Q214.G, Q215.G, Q216.G, Q217.G, Q218.G, R202.2, R203.1; no longer Q1.G, Q10.G, Q11.G, Q12.G, Q13.G, Q14.G, Q15.G, Q16.G, Q17.G, Q18.G, Q2.G, Q3.G, Q4.G, Q5.G, Q6.G, Q7.G, Q8.G, Q9.G, R32.2, R33.1
- net VCC: now also C1.2, C101.1, C201.1, C4.+, C5.1, IC101.DIR, IC101.VCC, IC201.DIR, IC201.VCC, IC4.OUTPUT_1, IC4.OUTPUT_2, IC5.DIR, IC5.VCC, R101.2, R102.1, R103.1, R6.1, R7.1, R8.1; no longer C10.+, C12.1, C14.1, C18.1, C8.2, IC11.OUTPUT_1, IC11.OUTPUT_2, IC12.DIR, IC12.VCC, IC6.DIR, IC6.VCC, IC7.DIR, IC7.VCC, R29.1, R31.1, R34.2, R37.1, R38.1, R39.1
- net VCCBUS: now also C2.1, C3.1, IC3.VCC, R101.1, R201.1; no longer C1.1, C9.1, IC5.VCC, R34.1, R35.1
- net VCCIO: now also C202.1, C203.1, C204.1, C205.1, C207.+, C210.1, IC202.VCC, IC203.VCC, Q201.S, Q202.S, Q203.S, Q204.S, Q205.S, Q206.S, Q207.S, Q208.S, Q209.S, Q210.S, Q211.S, Q212.S, Q213.S, Q214.S, Q215.S, Q216.S, Q217.S, Q218.S, R201.2, R202.1; no longer C13.1, C2.1, C23.1, C3.1, C30.1, C5.+, IC1.VCC, IC3.VCC, Q1.S, Q10.S, Q11.S, Q12.S, Q13.S, Q14.S, Q15.S, Q16.S, Q17.S, Q18.S, Q2.S, Q3.S, Q4.S, Q5.S, Q6.S, Q7.S, Q8.S, Q9.S, R32.1, R35.2
- net ZKEYB_RX: now also J1.3, RN1.8; no longer RN5.8, SV1.3
- net ZKEYB_TX_ORIG: now also J1.1, RN1.5; no longer RN5.5, SV1.1
Other:
- note added: "ACSI Logic Level Convertor"
- note added: "LEDs"
- note removed: "ACSI interface"
- note removed: "Logic Level Convertors & ACSI logic"
